File: schematics/Microbee_Kit_Main_Board/Microbee_Kit_Main_Board.kicad_sch (KiCad schematic)
At the start: 9 parts, among them U37 7805, X1 Core Board Connector 1, X4 Core Board Connector 2, X5 Power / Video / Cassette

Commit message: Continue with the main board schematic
Parts:
- added TP10, TP11: TestPoint, symbol Connector:TestPoint
Connections:
- net +5V: now also TP10.1
- net Earth: now also TP11.1
Other:
- added sheet Character Generation (character_generation.kicad_sch)
- added sheet IO Ports (io_ports.kicad_sch)
- added sheet Keyboard (keyboard.kicad_sch)
- added sheet Video Controller (video_controller.kicad_sch)
- added sheet Video Memory (video_memory.kicad_sch)
Changed lines of the file:
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@@
     (date "1982")
     (rev "1")
+    (comment 1 "(c) 1982 OJH MICROWORLD")
+    (comment 2 "Schematic Resrawn by Rhys Weatherley")
   )
   (junction (at 255.905 35.56) (diameter 0) (color 0 0 0 0)
@@
     (stroke (width 0) (type default))
   )
+  (wire (pts (xy 262.89 35.56) (xy 255.905 35.56))
+    (stroke (width 0) (type default))
+  )
   (wire (pts (xy 36.195 69.215) (xy 48.26 69.215))
     (stroke (width 0) (type default))
@@
   )
   (wire (pts (xy 36.195 104.775) (xy 48.26 104.775))
+    (stroke (width 0) (type default))
+  )
+  (wire (pts (xy 262.89 34.925) (xy 262.89 35.56))
     (stroke (width 0) (type default))
   )
@@
     )
   )
+  (symbol (lib_id "Connector:TestPoint") (at 262.89 34.925 0) (unit 1)
+    (in_bom yes) (on_board yes) (dnp no)
+    (property "Reference" "TP10" (at 260.35 29.21 0)
+      (effects (font (size 1.27 1.27)) (justify left))
+    )
+    (property "Value" "TestPoint" (at 265.43 32.893 0)
+      (effects (font (size 1.27 1.27)) (justify left) hide)
+    )
+    (property "Footprint" "" (at 267.97 34.925 0)
+      (effects (font (size 1.27 1.27)) hide)
+    )
+    (property "Datasheet" "~" (at 267.97 34.925 0)
+      (effects (font (size 1.27 1.27)) hide)
+    )
+    (pin "1")
+    (instances
+      (project "Microbee_Kit_Main_Board"
+        (path "/bb0ab0e6-f7d6-40cc-9fd3-11a13c259a53"
+          (reference "TP10") (unit 1)
+        )
+      )
+    )
+  )
   (symbol (lib_id "power:+10V") (at 71.755 64.77 0) (unit 1)
     (in_bom yes) (on_board yes) (dnp no) (fields_autoplaced)
@@
         (path "/bb0ab0e6-f7d6-40cc-9fd3-11a13c259a53"
           (reference "C30") (unit 1)
+        )
+      )
+    )
+  )
+  (symbol (lib_id "Connector:TestPoint") (at 269.24 34.925 0) (unit 1)
+    (in_bom yes) (on_board yes) (dnp no)
+    (property "Reference" "TP11" (at 266.7 29.21 0)
+      (effects (font (size 1.27 1.27)) (justify left))
+    )
+    (property "Value" "TestPoint" (at 271.78 32.893 0)
+      (effects (font (size 1.27 1.27)) (justify left) hide)
+    )
+    (property "Footprint" "" (at 274.32 34.925 0)
+      (effects (font (size 1.27 1.27)) hide)
+    )
+    (property "Datasheet" "~" (at 274.32 34.925 0)
+      (effects (font (size 1.27 1.27)) hide)
+    )
+    (pin "1")
+    (instances
+      (project "Microbee_Kit_Main_Board"
+        (path "/bb0ab0e6-f7d6-40cc-9fd3-11a13c259a53"
+          (reference "TP11") (unit 1)
         )
       )
@@
     )
   )
+  (symbol (lib_id "power:Earth") (at 269.24 34.925 0) (unit 1)
+    (in_bom yes) (on_board yes) (dnp no) (fields_autoplaced)
+    (property "Reference" "#PWR072" (at 269.24 41.275 0)
+      (effects (font (size 1.27 1.27)) hide)
+    )
+    (property "Value" "Earth" (at 269.24 38.735 0)
+      (effects (font (size 1.27 1.27)) hide)
+    )
+    (property "Footprint" "" (at 269.24 34.925 0)
+      (effects (font (size 1.27 1.27)) hide)
+    )
+    (property "Datasheet" "~" (at 269.24 34.925 0)
+      (effects (font (size 1.27 1.27)) hide)
+    )
+    (pin "1")
+    (instances
+      (project "Microbee_Kit_Main_Board"
+        (path "/bb0ab0e6-f7d6-40cc-9fd3-11a13c259a53"
+          (reference "#PWR072") (unit 1)
+        )
+      )
+    )
+  )
   (symbol (lib_id "Connector:DIN-5_180degree") (at 165.735 35.56 180) (unit 1)
     (in_bom yes) (on_board yes) (dnp no) (fields_autoplaced)
@@
     )
   )
-  (sheet (at 29.845 34.925) (size 24.765 12.7) (fields_autoplaced)
+  (sheet (at 179.07 99.695) (size 24.765 12.7) (fields_autoplaced)
     (stroke (width 0.1524) (type solid))
     (fill (color 0 0 0 0.0000))
-    (property "Sheetname" "CPU and Bus Tranceivers" (at 29.845 34.2134 0)
+    (property "Sheetname" "IO Ports" (at 179.07 98.9834 0)
       (effects (font (size 1.27 1.27)) (justify left bottom))
     )
-    (property "Sheetfile" "cpu_and_bus_tranceivers.kicad_sch" (at 29.845 48.2096 0)
+    (property "Sheetfile" "io_ports.kicad_sch" (at 179.07 112.9796 0)
       (effects (font (size 1.27 1.27)) (justify left top))
     )
@@
       )
     )
+  )
+  (sheet (at 223.52 77.47) (size 25.4 13.335) (fields_autoplaced)
+    (stroke (width 0.1524) (type solid))
+    (fill (color 0 0 0 0.0000))
+    (property "Sheetname" "Video Controller" (at 223.52 76.7584 0)
+      (effects (font (size 1.27 1.27)) (justify left bottom))
+    )
+    (property "Sheetfile" "video_controller.kicad_sch" (at 223.52 91.3896 0)
+      (effects (font (size 1.27 1.27)) (justify left top))
+    )
+    (instances
+      (project "Microbee_Kit_Main_Board"
+        (path "/bb0ab0e6-f7d6-40cc-9fd3-11a13c259a53" (page "5"))
+      )
+    )
+  )
+  (sheet (at 224.155 121.92) (size 24.13 12.7) (fields_autoplaced)
+    (stroke (width 0.1524) (type solid))
+    (fill (color 0 0 0 0.0000))
+    (property "Sheetname" "Character Generation" (at 224.155 121.2084 0)
+      (effects (font (size 1.27 1.27)) (justify left bottom))
+    )
+    (property "Sheetfile" "character_generation.kicad_sch" (at 224.155 135.2046 0)
+      (effects (font (size 1.27 1.27)) (justify left top))
+    )
+    (instances
+      (project "Microbee_Kit_Main_Board"
+        (path "/bb0ab0e6-f7d6-40cc-9fd3-11a13c259a53" (page "7"))
+      )
+    )
+  )
+  (sheet (at 179.07 121.92) (size 24.765 12.7) (fields_autoplaced)
+    (stroke (width 0.1524) (type solid))
+    (fill (color 0 0 0 0.0000))
+    (property "Sheetname" "Video Memory" (at 179.07 121.2084 0)
+      (effects (font (size 1.27 1.27)) (justify left bottom))
+    )
+    (property "Sheetfile" "video_memory.kicad_sch" (at 179.07 135.2046 0)
+      (effects (font (size 1.27 1.27)) (justify left top))
+    )
+    (instances
+      (project "Microbee_Kit_Main_Board"
+        (path "/bb0ab0e6-f7d6-40cc-9fd3-11a13c259a53" (page "4"))
+      )
+    )
+  )
+  (sheet (at 179.07 77.47) (size 24.765 12.7) (fields_autoplaced)
+    (stroke (width 0.1524) (type solid))
+    (fill (color 0 0 0 0.0000))
+    (property "Sheetname" "CPU and Bus Tranceivers" (at 179.07 76.7584 0)
+      (effects (font (size 1.27 1.27)) (justify left bottom))
+    )
+    (property "Sheetfile" "cpu_and_bus_tranceivers.kicad_sch" (at 179.07 90.7546 0)
+      (effects (font (size 1.27 1.27)) (justify left top))
+    )
+    (instances
+      (project "Microbee_Kit_Main_Board"
+        (path "/bb0ab0e6-f7d6-40cc-9fd3-11a13c259a53" (page "3"))
+      )
+    )
+  )
+  (sheet (at 224.155 99.06) (size 24.13 13.335) (fields_autoplaced)
+    (stroke (width 0.1524) (type solid))
+    (fill (color 0 0 0 0.0000))
+    (property "Sheetname" "Keyboard" (at 224.155 98.3484 0)
+      (effects (font (size 1.27 1.27)) (justify left bottom))
+    )
+    (property "Sheetfile" "keyboard.kicad_sch" (at 224.155 112.9796 0)
+      (effects (font (size 1.27 1.27)) (justify left top))
+    )
+    (instances
+      (project "Microbee_Kit_Main_Board"
+        (path "/bb0ab0e6-f7d6-40cc-9fd3-11a13c259a53" (page "6"))
+      )
+    )
