File: schematics/Microbee_Kit_Main_Board/character_generation.kicad_sch (KiCad schematic)
At the start: 8 parts, among them U10 74LS157, U12 74LS166, U13 2353, U14 74LS245, U18 6116, U21 74LS157, U6 74LS157

Commit message: Restoration and schematic updates
Parts:
- U13: value 2353 -> 2516
Changed lines of the file:
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@@
       (effects (font (size 1.27 1.27)) (justify left))
     )
-    (property "Value" "2353" (at 143.1641 54.61 0)
+    (property "Value" "2516" (at 143.1641 54.61 0)
       (effects (font (size 1.27 1.27)) (justify left))
     )
