File: schematics/Microbee_Kit_Main_Board/cpu_and_bus_tranceivers.kicad_sch (KiCad schematic)
At the start: 20 parts, among them U19 74LS245, U20 74LS02, U22 74LS244, U23 74LS04, U24 74LS244, U25 Z80CPU, U26 74LS161, U28 74LS244, U29 74LS00, U30 74LS27, U31 74LS04, U32 74LS92, U33 74C74

Commit message: Continue with the main board schematic
Parts:
- removed unit 3 of U20
- removed unit 2 of U20
- removed unit 1 of U20
- removed unit 3 of U31
- removed unit 4 of U31
- removed unit 1 of U33
- U33: footprint (none) -> Package_DIP:DIP-14_W7.62mm
Connections:
- net U33_PULLUP: now reaches RN3.10 (R9)
- no-connect marks 20 -> 19
Other:
- moved on the sheet: U31B
Changed lines of the file:
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@@
     (date "1982")
     (rev "1")
+    (comment 1 "(c) 1982 OJH MICROWORLD")
+    (comment 2 "Schematic Resrawn by Rhys Weatherley")
   )
   (junction (at 194.31 53.34) (diameter 0) (color 0 0 0 0)
@@
   (junction (at 208.28 138.43) (diameter 0) (color 0 0 0 0)
   )
-  (no_connect (at 161.925 177.165))
   (no_connect (at 90.17 151.765))
   (no_connect (at 154.305 177.165))
@@
   (no_connect (at 90.17 154.305))
   (no_connect (at 151.765 177.165))
-  (no_connect (at 27.94 78.105))
+  (no_connect (at 152.4 25.4))
   (no_connect (at 126.365 34.925))
   (no_connect (at 90.17 149.225))
   (no_connect (at 195.58 151.13))
   (no_connect (at 90.17 146.685))
-  (no_connect (at 43.18 78.105))
+  (no_connect (at 167.64 25.4))
   (no_connect (at 126.365 32.385))
   (bus_entry (at 19.05 184.785) (size 2.54 2.54)
@@
     (stroke (width 0) (type default))
   )
+  (wire (pts (xy 161.925 173.99) (xy 161.925 177.165))
+    (stroke (width 0) (type default))
+  )
   (wire (pts (xy 182.88 58.42) (xy 182.88 30.48))
     (stroke (width 0) (type default))
@@
     )
   )
+  (global_label "U33_PULLUP" (shape input) (at 161.925 173.99 90) (fields_autoplaced)
+    (effects (font (size 1.27 1.27)) (justify left))
+    (property "Intersheetrefs" "${INTERSHEET_REFS}" (at 161.925 159.0305 90)
+      (effects (font (size 1.27 1.27)) (justify left) hide)
+    )
+  )
   (global_label "~{ROM_SEL}" (shape input) (at 27.305 116.205 180) (fields_autoplaced)
     (effects (font (size 1.27 1.27)) (justify right))
@@
     )
   )
-  (symbol (lib_id "74xx:74LS02") (at 318.135 136.525 0) (unit 3)
-    (in_bom yes) (on_board yes) (dnp no) (fields_autoplaced)
-    (property "Reference" "U20" (at 318.135 128.27 0)
-      (effects (font (size 1.27 1.27)))
-    )
-    (property "Value" "74LS02" (at 318.135 130.81 0)
-      (effects (font (size 1.27 1.27)))
-    )
-    (property "Footprint" "" (at 318.135 136.525 0)
-      (effects (font (size 1.27 1.27)) hide)
-    )
-    (property "Datasheet" "http://www.ti.com/lit/gpn/sn74ls02" (at 318.135 136.525 0)
-      (effects (font (size 1.27 1.27)) hide)
-    )
-    (pin "13")
-    (pin "11")
-    (pin "12")
-    (pin "8")
-    (pin "7")
-    (pin "10")
-    (pin "9")
-    (pin "5")
-    (pin "14")
-    (pin "2")
-    (pin "3")
-    (pin "6")
-    (pin "4")
-    (pin "1")
-    (instances
-      (project "Microbee_Kit_Main_Board"
-        (path "/bb0ab0e6-f7d6-40cc-9fd3-11a13c259a53/d3ef44f1-c26e-4383-92de-6831636e332e"
-          (reference "U20") (unit 3)
-        )
-      )
-    )
-  )
   (symbol (lib_id "power:Earth") (at 208.28 60.96 0) (unit 1)
     (in_bom yes) (on_board yes) (dnp no) (fields_autoplaced)
@@
     )
   )
-  (symbol (lib_id "74xx:74LS04") (at 35.56 78.105 0) (unit 2)
+  (symbol (lib_id "74xx:74LS04") (at 160.02 25.4 0) (unit 2)
     (in_bom yes) (on_board yes) (dnp no) (fields_autoplaced)
-    (property "Reference" "U31" (at 35.56 69.215 0)
+    (property "Reference" "U31" (at 160.02 16.51 0)
       (effects (font (size 1.27 1.27)))
     )
-    (property "Value" "74LS04" (at 35.56 71.755 0)
+    (property "Value" "74LS04" (at 160.02 19.05 0)
       (effects (font (size 1.27 1.27)))
     )
-    (property "Footprint" "" (at 35.56 78.105 0)
+    (property "Footprint" "" (at 160.02 25.4 0)
       (effects (font (size 1.27 1.27)) hide)
     )
-    (property "Datasheet" "http://www.ti.com/lit/gpn/sn74LS04" (at 35.56 78.105 0)
+    (property "Datasheet" "http://www.ti.com/lit/gpn/sn74LS04" (at 160.02 25.4 0)
       (effects (font (size 1.27 1.27)) hide)
     )
@@
       (effects (font (size 1.27 1.27)) (justify left))
     )
-    (property "Footprint" "" (at 31.115 126.365 0)
+    (property "Footprint" "Package_DIP:DIP-14_W7.62mm" (at 31.115 126.365 0)
       (effects (font (size 1.27 1.27)) hide)
     )
@@
       (effects (font (size 1.27 1.27)) (justify left))
     )
-    (property "Footprint" "" (at 272.415 78.105 0)
+    (property "Footprint" "Package_DIP:DIP-14_W7.62mm" (at 272.415 78.105 0)
       (effects (font (size 1.27 1.27)) hide)
     )
@@
     )
   )
-  (symbol (lib_id "74xx:74LS02") (at 316.865 115.57 0) (unit 2)
-    (in_bom yes) (on_board yes) (dnp no) (fields_autoplaced)
-    (property "Reference" "U20" (at 316.865 106.68 0)
-      (effects (font (size 1.27 1.27)))
-    )
-    (property "Value" "74LS02" (at 316.865 109.22 0)
-      (effects (font (size 1.27 1.27)))
-    )
-    (property "Footprint" "" (at 316.865 115.57 0)
-      (effects (font (size 1.27 1.27)) hide)
-    )
-    (property "Datasheet" "http://www.ti.com/lit/gpn/sn74ls02" (at 316.865 115.57 0)
-      (effects (font (size 1.27 1.27)) hide)
-    )
-    (pin "13")
-    (pin "11")
-    (pin "12")
-    (pin "8")
-    (pin "7")
-    (pin "10")
-    (pin "9")
-    (pin "5")
-    (pin "14")
-    (pin "2")
-    (pin "3")
-    (pin "6")
-    (pin "4")
-    (pin "1")
-    (instances
-      (project "Microbee_Kit_Main_Board"
-        (path "/bb0ab0e6-f7d6-40cc-9fd3-11a13c259a53/d3ef44f1-c26e-4383-92de-6831636e332e"
-          (reference "U20") (unit 2)
-        )
-      )
-    )
-  )
-  (symbol (lib_id "74xx:74LS04") (at 360.045 39.37 0) (unit 3)
-    (in_bom yes) (on_board yes) (dnp no) (fields_autoplaced)
-    (property "Reference" "U31" (at 360.045 30.48 0)
-      (effects (font (size 1.27 1.27)))
-    )
-    (property "Value" "74LS04" (at 360.045 33.02 0)
-      (effects (font (size 1.27 1.27)))
-    )
-    (property "Footprint" "" (at 360.045 39.37 0)
-      (effects (font (size 1.27 1.27)) hide)
-    )
-    (property "Datasheet" "http://www.ti.com/lit/gpn/sn74LS04" (at 360.045 39.37 0)
-      (effects (font (size 1.27 1.27)) hide)
-    )
-    (pin "13")
-    (pin "5")
-    (pin "12")
-    (pin "9")
-    (pin "14")
-    (pin "4")
-    (pin "10")
-    (pin "3")
-    (pin "1")
-    (pin "2")
-    (pin "8")
-    (pin "7")
-    (pin "11")
-    (pin "6")
-    (instances
-      (project "Microbee_Kit_Main_Board"
-        (path "/bb0ab0e6-f7d6-40cc-9fd3-11a13c259a53/d3ef44f1-c26e-4383-92de-6831636e332e"
-          (reference "U31") (unit 3)
-        )
-      )
-    )
-  )
   (symbol (lib_id "power:Earth") (at 258.445 90.805 0) (unit 1)
     (in_bom yes) (on_board yes) (dnp no) (fields_autoplaced)
@@
     )
   )
-  (symbol (lib_id "74xx:74LS02") (at 318.135 99.695 0) (unit 1)
-    (in_bom yes) (on_board yes) (dnp no) (fields_autoplaced)
-    (property "Reference" "U20" (at 318.135 91.44 0)
-      (effects (font (size 1.27 1.27)))
-    )
-    (property "Value" "74LS02" (at 318.135 93.98 0)
-      (effects (font (size 1.27 1.27)))
-    )
-    (property "Footprint" "" (at 318.135 99.695 0)
-      (effects (font (size 1.27 1.27)) hide)
-    )
-    (property "Datasheet" "http://www.ti.com/lit/gpn/sn74ls02" (at 318.135 99.695 0)
-      (effects (font (size 1.27 1.27)) hide)
-    )
-    (pin "13")
-    (pin "11")
-    (pin "12")
-    (pin "8")
-    (pin "7")
-    (pin "10")
-    (pin "9")
-    (pin "5")
-    (pin "14")
-    (pin "2")
-    (pin "3")
-    (pin "6")
-    (pin "4")
-    (pin "1")
-    (instances
-      (project "Microbee_Kit_Main_Board"
-        (path "/bb0ab0e6-f7d6-40cc-9fd3-11a13c259a53/d3ef44f1-c26e-4383-92de-6831636e332e"
-          (reference "U20") (unit 1)
-        )
-      )
-    )
-  )
   (symbol (lib_id "74xx:74LS00") (at 258.445 41.275 0) (unit 5)
     (in_bom yes) (on_board yes) (dnp no)
@@
     )
   )
-  (symbol (lib_id "74xx:74LS04") (at 360.045 48.895 0) (unit 4)
-    (in_bom yes) (on_board yes) (dnp no) (fields_autoplaced)
-    (property "Reference" "U31" (at 360.045 40.64 0)
-      (effects (font (size 1.27 1.27)))
-    )
-    (property "Value" "74LS04" (at 360.045 43.18 0)
-      (effects (font (size 1.27 1.27)))
-    )
-    (property "Footprint" "" (at 360.045 48.895 0)
-      (effects (font (size 1.27 1.27)) hide)
-    )
-    (property "Datasheet" "http://www.ti.com/lit/gpn/sn74LS04" (at 360.045 48.895 0)
-      (effects (font (size 1.27 1.27)) hide)
-    )
-    (pin "13")
-    (pin "5")
-    (pin "12")
-    (pin "9")
-    (pin "14")
-    (pin "4")
-    (pin "10")
-    (pin "3")
-    (pin "1")
-    (pin "2")
-    (pin "8")
-    (pin "7")
-    (pin "11")
-    (pin "6")
-    (instances
-      (project "Microbee_Kit_Main_Board"
-        (path "/bb0ab0e6-f7d6-40cc-9fd3-11a13c259a53/d3ef44f1-c26e-4383-92de-6831636e332e"
-          (reference "U31") (unit 4)
-        )
-      )
-    )
-  )
   (symbol (lib_id "power:+5V") (at 240.665 120.65 0) (unit 1)
     (in_bom yes) (on_board yes) (dnp no) (fields_autoplaced)
@@
         )
       )
-    )
-  )
-  (symbol (lib_id "74xx:74LS74") (at 364.49 151.765 0) (unit 1)
-    (in_bom yes) (on_board yes) (dnp no) (fields_autoplaced)
-    (property "Reference" "U33" (at 366.6841 142.24 0)
-      (effects (font (size 1.27 1.27)) (justify left))
-    )
-    (property "Value" "74C74" (at 366.6841 144.78 0)
-      (effects (font (size 1.27 1.27)) (justify left))
-    )
-    (property "Footprint" "" (at 364.49 151.765 0)
-      (effects (font (size 1.27 1.27)) hide)
-    )
-    (property "Datasheet" "74xx/74hc_hct74.pdf" (at 364.49 151.765 0)
-      (effects (font (size 1.27 1.27)) hide)
-    )
-    (pin "4")
-    (pin "5")
-    (pin "6")
-    (pin "3")
-    (pin "8")
-    (pin "7")
-    (pin "13")
-    (pin "10")
-    (pin "11")
-    (pin "12")
-    (pin "14")
-    (pin "9")
-    (pin "1")
-    (pin "2")
-    (instances
-      (project "Microbee_Kit_Main_Board"
-        (path "/bb0ab0e6-f7d6-40cc-9fd3-11a13c259a53/d3ef44f1-c26e-4383-92de-6831636e332e"
-          (reference "U33") (unit 1)
-        )
-      )

Commit message: Restoration and schematic updates
Connections:
- net 12MHz: now also U26.2 (CP)
- net CLOCK: no longer U26.2 (CP)
Other:
- note added: "1.5MHz"
Changed lines of the file:
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@@
+    (effects (font (size 1.27 1.27)) (justify left bottom))
+  )
+  (text "1.5MHz" (at 126.365 166.37 0)
     (effects (font (size 1.27 1.27)) (justify left bottom))
   )
@@
     )
   )
-  (global_label "CLOCK" (shape input) (at 81.915 167.005 180) (fields_autoplaced)
-    (effects (font (size 1.27 1.27)) (justify right))
-    (property "Intersheetrefs" "${INTERSHEET_REFS}" (at 72.7612 167.005 0)
-      (effects (font (size 1.27 1.27)) (justify right) hide)
-    )
+  (global_label "12MHz" (shape input) (at 81.915 167.005 180) (fields_autoplaced)
+    (effects (font (size 1.27 1.27)) (justify right))
+    (property "Intersheetrefs" "${INTERSHEET_REFS}" (at 72.7008 167.005 0)
+      (effects (font (size 1.27 1.27)) (justify right) hide)
+    )
