File: schematics/Microbee_Kit_Main_Board/video_controller.kicad_sch (KiCad schematic)
At the start: 18 parts, among them Q2 BC547, U11 74LS245, U15 74LS175, U17 74LS86, U20 74LS02, U9 6545-1

Commit message: Restoration and schematic updates
Other:
- note added: "1.5MHz"
- note added: "30Hz"
- note added: "5.8557kHz"
Changed lines of the file:
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@@
     (stroke (width 0) (type default))
+  )
+  (text "1.5MHz" (at 111.125 73.025 0)
+    (effects (font (size 1.27 1.27)) (justify left bottom))
+  )
+  (text "5.8557kHz" (at 166.37 103.505 0)
+    (effects (font (size 1.27 1.27)) (justify left bottom))
+  )
+  (text "30Hz" (at 171.45 111.125 0)
+    (effects (font (size 1.27 1.27)) (justify left bottom))
   )
   (label "MA13" (at 168.91 81.915 0) (fields_autoplaced)
