File: schematics/Microbee_Kit_Main_Board/keyboard.kicad_sch (KiCad schematic)
At the start: 63 parts, among them SW1 @, SW10 Q, SW11 Y, SW12 1, SW13 9, SW14 BS, SW15 B, SW16 J, SW17 R, SW18 Z, SW19 2, SW2 H, SW20 *, SW21 TAB, SW22 C, SW23 K, SW24 S, SW25 [, SW26 3, SW27 +, SW28 LF, SW29 D, SW3 P, SW30 L, SW31 T, SW32 \, SW33 4, SW34 <, SW35 CR, SW36 E, SW37 M, SW38 U, SW39 ], SW4 X, SW40 5, SW41 =, SW42 LOCK, SW43 F, SW44 N, SW45 V, SW46 ^, SW47 6, SW48 >, SW49 BRK, SW5 0, SW50 G, SW51 O, SW52 W, SW53 DEL, SW54 7, SW55 /, SW56 SP, SW57 CTRL, SW58 LSHIFT, SW59 RSHIFT, SW6 8, SW7 ESC, SW8 A, SW9 I, U20 74LS02, U4 74LS151, U7 74LS156

Commit message: Continue documenting the restoration
Other:
- note removed: "TBD: REPT key?"
Changed lines of the file:
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@@
     (stroke (width 0) (type default))
-  )
-  (text "TBD: REPT key?" (at 230.505 126.365 0)
-    (effects (font (size 1.27 1.27)) (justify left bottom))
   )
   (text "TBD: Connections to Video Controller Schematic" (at 40.64 26.67 0)
