File: schematics/Microbee_Kit_Core_Board/ram_bank_1.kicad_sch (KiCad schematic)
At the start: 24 parts, among them U1 6116, U10 6116, U11 4053, U12 6116, U2 74LS138, U3 6116, U32 74LS04, U4 4053, U5 6116, U6 6116, U7 4053, U8 6116, U9 6116

Commit message: Restoration and schematic updates
Connections:
- net +5V renamed VMEM
Other:
- note added: "$0000"
- note added: "$0800"
- note added: "$1000"
- note added: "$1800"
- note added: "$2000"
- note added: "$2800"
- note added: "$3000"
- note added: "$3800"
