File: schematics/Microbee_Kit_Core_Board/ram_bank_2.kicad_sch (KiCad schematic)
At the start: 21 parts, among them U13 6116, U14 74LS138, U15 6116, U16 4053, U17 6116, U18 6116, U19 4053, U20 6116, U21 6116, U22 6116, U23 4053, U24 6116

Commit message: Restoration and schematic updates
Connections:
- net +5V renamed VMEM
Other:
- note added: "$4000"
- note added: "$4800"
- note added: "$5000"
- note added: "$5800"
- note added: "$6000"
- note added: "$6800"
- note added: "$7000"
- note added: "$7800"
