File: schematics/Microbee_Kit_Core_Board/rom_bank.kicad_sch (KiCad schematic)
At the start: 15 parts, among them U25 2532, U26 74LS138, U27 2532, U28 2532, U30 2532, U31 2532, U33 2532, U34 2532

Commit message: Restoration and schematic updates
Other:
- note added: "$8000"
- note added: "$9000"
- note added: "$A000"
- note added: "$B000"
- note added: "$C000"
- note added: "$D000"
- note added: "$E000"
Changed lines of the file:
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@@
     (stroke (width 0) (type default))
+  )
+  (text "$B000" (at 233.045 36.195 0)
+    (effects (font (size 1.27 1.27)) (justify left bottom))
   )
   (text "$8000 - $BFFF BASIC ROM's\n$C000 - $DFFF EDASM ROM's\n$E000 - $EFFF NET ROM"
     (at 236.22 100.965 0)
+    (effects (font (size 1.27 1.27)) (justify left bottom))
+  )
+  (text "$8000" (at 102.87 36.195 0)
+    (effects (font (size 1.27 1.27)) (justify left bottom))
+  )
+  (text "$E000" (at 189.865 85.725 0)
+    (effects (font (size 1.27 1.27)) (justify left bottom))
+  )
+  (text "$9000" (at 146.685 36.195 0)
     (effects (font (size 1.27 1.27)) (justify left bottom))
   )
@@
     (effects (font (size 1.27 1.27)) (justify left bottom))
   )
+  (text "$D000" (at 146.685 85.725 0)
+    (effects (font (size 1.27 1.27)) (justify left bottom))
+  )
+  (text "$A000" (at 189.865 36.195 0)
+    (effects (font (size 1.27 1.27)) (justify left bottom))
+  )
+  (text "$C000" (at 102.87 85.725 0)
+    (effects (font (size 1.27 1.27)) (justify left bottom))
+  )
