File: schematics/Microbee_Kit_Core_Board/Microbee_Kit_Core_Board.kicad_sch (KiCad schematic)
At the start: 28 parts, among them Q1 BC558, U29 MC14584B, U35 LM7805, X1 Main Board Connector 1, X2 Expansion Connector, X3 Main Board Connector 2, X4 3V, X5 0V

Commit message: Restoration and schematic updates
Connections:
- net SUPPLY renamed VMEM
Changed lines of the file:
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@@
   (junction (at 109.855 106.68) (diameter 0) (color 0 0 0 0)
+  )
+  (junction (at 218.44 109.855) (diameter 0) (color 0 0 0 0)
   )
   (junction (at 111.76 111.125) (diameter 0) (color 0 0 0 0)
@@
   )
   (wire (pts (xy 97.155 75.565) (xy 109.22 75.565))
+    (stroke (width 0) (type default))
+  )
+  (wire (pts (xy 218.44 107.315) (xy 218.44 109.855))
     (stroke (width 0) (type default))
   )
@@
         )
       )
+    )
+  )
+  (symbol (lib_id "power:VMEM") (at 218.44 107.315 0) (unit 1)
+    (in_bom yes) (on_board yes) (dnp no) (fields_autoplaced)
+    (property "Reference" "#PWR0156" (at 218.44 111.125 0)
+      (effects (font (size 1.27 1.27)) hide)
+    )
+    (property "Value" "VMEM" (at 218.44 102.235 0)
+      (effects (font (size 1.27 1.27)))
+    )
+    (property "Footprint" "" (at 218.44 107.315 0)
+      (effects (font (size 1.27 1.27)) hide)
+    )
+    (property "Datasheet" "" (at 218.44 107.315 0)
+      (effects (font (size 1.27 1.27)) hide)
+    )
+    (pin "1")
+    (instances
+      (project "Microbee_Kit_Core_Board"
+        (path "/fd592533-bded-4397-9d77-d2c17ab5a48c"
+          (reference "#PWR0156") (unit 1)
+        )
+      )

Commit message: Continue documenting the restoration
Parts:
- LED1: value 5V Power -> Backup
Changed lines of the file:
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@@
       (effects (font (size 1.27 1.27)) (justify right))
     )
-    (property "Value" "5V Power" (at 271.78 147.0025 90)
+    (property "Value" "Backup" (at 271.78 147.0025 90)
       (effects (font (size 1.27 1.27)) (justify right))
     )
